File: Hardware/Eagle Files/OBD-Interface/OBD-Schematic.sch (EAGLE design)
At the start: 0 parts

Commit message: LTC3633 Wired Up
Added the LTC3633 Buck switching PSU.
Parts:
- added C1: (no value), adafruit:C-USC0805
- added C2: 22uG, adafruit:C-USC0805
- added C3, C6: 0.1uF, adafruit:C-USC0805
- added C4: 22uF, adafruit:C-USC0805
- added L1: 1.5uH, rcl:L-USL5650M
- added L2: 1uF, rcl:L-USL5650M
- added R1: 73.2k, adafruit:R-US_R0805
- added R2, R4: 10k, adafruit:R-US_R0805
- added R3: 45.3k, adafruit:R-US_R0805
- added U1: LTC3633EUFDPBF, LTC_By_element14_Batch_1:LTC3633EUFDPBF
Connections:
- new net +12V: C1.1, U1.RUN1, U1.RUN2, U1.VIN1, U1.VIN1_2, U1.VIN2, U1.VIN2_2
- new net +3V3: C4.1, L2.1, R3.1, U1.VON1
- new net +5V: C2.1, L1.1, R1.1, U1.VON2
- new net BOOST1: C6.1, U1.BOOST1
- new net BOOST2: C3.1, U1.BOOST2
- new net GND: C1.2, C2.2, C4.2, R2.2, R4.2, U1.EP, U1.INTVCC, U1.ITH1, U1.ITH2, U1.MODE/SYNC, U1.PHMODE, U1.RT, U1.SGND, U1.V2P5
- new net SW1: C6.2, L2.2, U1.SW1, U1.SW1_2
- new net SW2: C3.2, L1.2, U1.SW2, U1.SW2_2
- new net VFB1: R3.2, R4.1, U1.VFB1
- new net VFB2: R1.2, R2.1, U1.VFB2
