File: Hardware/Eagle Files/OBD-Interface/OBD-Schematic.sch (EAGLE design)
At the start: 12 parts, among them U1 LTC3633EUFDPBF

Commit message: J1850VPW Interface hardware
Hardware to interface between the micro and the bus laid. Needs to be
valued.
Parts:
- added C5, C7, C8, C9: (no value), adafruit:C-USC0805
- added D1, D2: (no value), adafruit:DIODESOT23_REFLOW
- added LED1: (no value), adafruit:LEDCHIP-LED0805
- added Q1, Q2: BSS138, SparkFun-DiscreteSemi:MOSFET-NCHANNELBSS123LT1G
- added Q3: ZXMP6A13FTA, SparkFun-DiscreteSemi:MOSFET-NCHANNELBSS123LT1G
- added R10, R11, R12, R13, R14, R5, R6, R7, R8, R9: (no value), adafruit:R-US_R0805
- added U$1: ATSAM4C32, atmel:ATSAM4C32
- added U2: V_REG_317DPACK, SparkFun-PowerIC:V_REG_317DPACK
- added U3: LM339, SparkFun-AnalogIC:LM339
Connections:
- new net !VPW_RX: R14.1, U3B.OUT
- new net 2.8V: Q3.S, R9.2
- new net 5/7V: C8.1, R5.2, R8.2, U2.OUT
- new net J1850BUS+: D1.C, R10.2, R11.1
- new net J1850BUS+_TX: Q2.G
- new net N$1: C7.1, U$1G$1.VDDCORE@11, U$1G$1.VDDCORE@44, U$1G$1.VDDCORE@63, U$1G$1.VDDCORE@89, U$1G$1.VDDOUT@86, U$1G$1.VDDPLL@53
- new net N$10: D2.A, R10.1
- new net N$13: LED1.A, R8.1
- new net N$2: C5.1, U$1G$1.VDDLCD@92
- new net N$3: Q1.S, R6.1, R7.2
- new net N$4: Q2.S, Q3.G, R9.1
- new net N$5: R12.1, R13.2, U3B.+IN
- new net N$7: R5.1, R6.2, U2.ADJ
- new net N$8: D1.A, Q3.D
- new net N$9: R11.2, U3B.-IN
- new net PWM/!VPW: Q1.G
- new net VBAT: C9.1, U2.IN
- net +3V3: now also R14.2, U$1G$1.VDDBU@34, U$1G$1.VDDIN@85, U$1G$1.VDDIO@33, U$1G$1.VDDIO@49, U$1G$1.VDDIO@76, U$1G$1.VDDIO@99
- net +5V: now also R12.2
- net GND: now also C5.2, C7.2, C8.2, C9.2, D2.C, LED1.C, Q1.D, Q2.D, R13.1, R7.1, U$1G$2.GND@4, U$1G$2.GND@42, U$1G$2.GND@52, U$1G$2.GND@78
Other:
- note added: "J1850 VPW TX"
- note added: "Selectable 5.76V or 7.71V"

Commit message: CAN Transceiver Added
Everything needs to be valued. This completes the GM side of the
transceiver. v1 will only talk to GM. This is where the market is
currently and I know the most about. Future revisions will add support
for ISO and J1850 PWM
Parts:
- added C10, C11, C12: (no value), adafruit:C-USC0805
- added R15, R16, R17: (no value), adafruit:R-US_R0805
- added U4: MCP2551, SparkFun-DigitalIC:MCP2551
- Q3: device SparkFun-DiscreteSemi:MOSFET-NCHANNELBSS123LT1G -> SparkFun-DiscreteSemi:MOSFET-PCHANNEL
Connections:
- new net CAN_HI: R16.1, U4.CANH
- new net CAN_LO: R15.1, U4.CANL
- new net CAN_RX: U4.RXD
- new net CAN_TX: U4.TXD
- new net N$14: C10.1, R15.2
- new net N$15: C11.1, R16.2
- new net N$6: Q2.D, Q3.G, R9.1
- net +5V: now also C12.1, U4.VDD
- net 2.8V: now also Q3.D; no longer Q3.S
- net GND: now also C10.2, C11.2, C12.2, Q2.S, R17.2, U4.VSS; no longer Q2.D
- net N$4: now also R17.1, U4.RS; no longer Q2.S, Q3.G, R9.1
- net N$8: now also Q3.S; no longer Q3.D
Other:
- note added: "CAN Transceiver"
- note added: "J1850 VPW RX"
- moved on the sheet: Q2, Q3

Commit message: Added the SAM4C (in the 144-pin package) to the schematic and started hooking it up.
Parts:
- added C13, C19: 10 uF, passives:C0603
- added C14, C15, C16, C17, C18, C20, C24, C26, C27, C28, C29: 100 nF, passives:C0603
- added C21, C22: 18 pF, passives:C0603
- added C23, C25: 2.2 uF, passives:C0603
- added JP1: (no value), SparkFun-Connectors:M10X2
- added R18, R19, R20, R21, R22: 100k, passives:R0603
- added R23: 0 (NOPOP), passives:R0603
- added Y1: 32.768 kHz, adafruit:CRYSTALSM49
- C5: value (none) -> 10 uF; device adafruit:C-USC0805 -> passives:C0603
- C7: value (none) -> 100 nF; device adafruit:C-USC0805 -> passives:C0603
- U$1: value ATSAM4C32 -> SAM4C32C-144; device atmel:ATSAM4C32 -> OBD-Interface:SAM4C32C-144
Connections:
- removed net N$2: C5.1, U$1G$1.VDDLCD@92
- new net N$11: C22.2, U$1G$1.XIN32, Y1.1
- new net N$12: C21.2, U$1G$1.XOUT32, Y1.2
- new net N$19: JP1.15, R23.1
- new net NRST: R22.1, R23.2, U$1G$1.NRST
- new net TCK: JP1.11, JP1.9, R21.1, U$1G$3.PB3/TCK/SWCLK
- new net TDI: JP1.5, R19.1, U$1G$3.PB0/TWD1/TDI
- new net TDO: JP1.13, U$1G$3.PB1/TWCK1/TDO/TRACESWO
- new net TMS: JP1.7, R20.1, U$1G$3.PB2/TMS/SWDIO
- new net VDDLCD: C19.1, C20.1, U$1G$1.VDDLCD
- new net VDDOUT: C23.1, C24.1, C25.1, C26.1, C27.1, C28.1, C29.1, U$1G$1.VDDCORE, U$1G$1.VDDOUT, U$1G$1.VDDPLL
- net +3V3: now also C13.1, C14.1, C15.1, C16.1, C17.1, C18.1, C5.1, C7.1, JP1.1, JP1.2, R18.2, R19.2, R20.2, R21.2, R22.2, U$1G$1.VDDBU, U$1G$1.VDDIN, U$1G$1.VDDIO; no longer U$1G$1.VDDBU@34, U$1G$1.VDDIN@85, U$1G$1.VDDIO@33, U$1G$1.VDDIO@49, U$1G$1.VDDIO@76, U$1G$1.VDDIO@99
- net GND: now also C13.2, C14.2, C15.2, C16.2, C17.2, C18.2, C19.2, C20.2, C21.1, C22.1, C23.2, C24.2, C25.2, C26.2, C27.2, C28.2, C29.2, JP1.10, JP1.12, JP1.14, JP1.16, JP1.18, JP1.20, JP1.4, JP1.6, JP1.8, U$1G$1.GND; no longer U$1G$2.GND@4, U$1G$2.GND@42, U$1G$2.GND@52, U$1G$2.GND@78
- net N$1: now also JP1.3, R18.1; no longer C7.1, U$1G$1.VDDCORE@11, U$1G$1.VDDCORE@44, U$1G$1.VDDCORE@63, U$1G$1.VDDCORE@89, U$1G$1.VDDOUT@86, U$1G$1.VDDPLL@53
Other:
- note added: "NC"
- note added: "Note: EK has filtering on VDDPLL."
- note added: "VDDBU: 100 nF"
- note added: "VDDCORE: 2.2 uF 100 nF x4"
- note added: "VDDIN: 10 uF 100 nF"
- note added: "VDDIO: 10 uF 100 nF x4"
- note added: "VDDLCD: 2.2uF 100nF"
- note added: "VDDOUT: 2.2 uF 100 nF"

Commit message: Added OBD header and uSD Card slot
Parts:
- added C30: 0.1uF, SparkFun-Capacitors:0.1UF-25V(+80/-20%)(0603)
- added JP2: (no value), SparkFun-Connectors:M08X2
- added R24, R25, R26, R27: 3.3K, SparkFun-Resistors:3.3KOHM1/10W1%(0603)
- added U5: USD-SOCKETUSD, SparkFun-Connectors:USD-SOCKETUSD
Connections:
- new net N$20: C30.1, U5.CD2, U5.GND, U5.SHIELD@3
- new net SD_SPI_CS: R24.1, U$1G$2.PA5/AD2, U5.CS
- new net SD_SPI_DI: R26.1, U$1G$2.PA7, U5.DI
- new net SD_SPI_DO: R25.1, U$1G$2.PA6, U5.DO
- new net SD_SPI_SCK: R27.1, U$1G$2.PA8, U5.SCK
- net +12V: now also JP2.16
- net +3V3: now also U5.VCC
- net CAN_HI: now also JP2.6
- net CAN_LO: now also JP2.14
- net GND: now also C30.2, R24.2, R25.2, R26.2, R27.2
- net J1850BUS+: now also JP2.2
Other:
- note added: "CLEAN UP"
- note added: "Mirco-SD Card Interface"
- note added: "OBD Header"

Commit message: Added Flash and 8Mhz oscillator
Parts:
- removed R26, R27: 3.3K, SparkFun-Resistors:3.3KOHM1/10W1%(0603)
- added C31: (no value), passives:C0603
- added C32, C33: 18pF, passives:C0603
- added IC3: MS25P05-A, OBD-Interface:MS25P05-A
- added Y2CTX900-ND: 8 Mhz, SparkFun-FreqCtrl:CRYSTALHC49US
- R24, R25: value 3.3K -> 0R; device SparkFun-Resistors:3.3KOHM1/10W1%(0603) -> passives:R0603
- renumbered U1 to IC1, U2 to IC4, U4 to IC5
Connections:
- new net FLASH_CS: IC3.CS, U$1G$4.PC2
- new net FLASH_HLD: IC3.HLD, U$1G$4.ERASE/PC9
- new net FLASH_MISO: IC3.MISO, U$1G$4.PC3
- new net FLASH_MOSI: IC3.MOSI, U$1G$4.PC4
- new net FLASH_SCLK: IC3.SCLK
- new net FLASH_SPCK: U$1G$4.PC5
- new net FLASH_WP: IC3.WP, U$1G$4.PC8
- new net N$16: R24.1, U$1G$2.PA29
- new net N$17: R25.1, U$1G$2.PA31
- new net N$18: C33.2, R25.2, Y2CTX900-ND.1
- new net N$21: C31.2, IC3.VSS
- new net N$22: C32.2, R24.2, Y2CTX900-ND.2
- net +3V3: now also IC3.VCC
- net GND: now also C31.1, C32.1, C33.1; no longer R24.2, R25.2, R26.2, R27.2
- net SD_SPI_CS: no longer R24.1
- net SD_SPI_DI: no longer R26.1
- net SD_SPI_DO: no longer R25.1
- net SD_SPI_SCK: no longer R27.1
Other:
- note added: "M25P05-AVMN6TP FLASH"
- note added: "NOTE: May need filtering here? VBatt (From OBD) can fluctuate between 8-16V in extreme cases"
- moved on the sheet: C30, JP2, U5

Commit message: Added USB, Debug Header, Added Board File.
Parts:
- removed C30: 0.1uF, SparkFun-Capacitors:0.1UF-25V(+80/-20%)(0603)
- removed C31: (no value), passives:C0603
- removed U$1: SAM4C32C-144, OBD-Interface:SAM4C32C-144
- added C36: 10nF, passives:C0603
- added C37, C38: 47pF, passives:C0603
- added C39: 0.1uF, passives:C0603
- added IC2: FT232RL, OBD-Interface:FT232RL
- added JP3: (no value), adafruit:PINHD-1X6CLEAN
- added LED2, LED3: (no value), adafruit:LEDCHIPLED_0805
- added R26, R27: 330R, passives:R0603
- added U$3: SAM4C32C-100, OBD-Interface:SAM4C32C-100
- added X1: MINI-USB_SHIELD5P2-32005-601, con-cypressindustries:MINI-USB_SHIELD5P2-32005-601
Connections:
- removed net FLASH_SPCK: U$1G$4.PC5
- removed net N$20: C30.1, U5.CD2, U5.GND, U5.SHIELD@3
- removed net N$21: C31.2, IC3.VSS
- new net N$25: C37.1, IC2.USBDM, X1G41.2
- new net N$26: C38.2, IC2.USBDP, X1G41.3
- new net N$27: LED2.A, R26.1
- new net N$28: LED3.A, R27.1
- new net N$29: IC2.CBUS0, LED2.C
- new net N$30: IC2.CBUS1, LED3.C
- new net N$31: JP3.1, U$3G$3.PB6
- new net N$32: JP3.2, U$3G$3.PB13/AD3
- new net N$33: C39.1, IC2.3V3OUT
- new net N$34: JP3.3, U$3G$3.PB14
- new net N$35: JP3.4, U$3G$3.PB15
- new net N$36: JP3.5, U$3G$3.PB16
- new net N$37: JP3.6, U$3G$3.PB17
- new net SLEEP: IC2.CBUS4
- new net UART_RX: IC2.RXD, U$3G$3.PB4
- new net UART_TX: IC2.TXD, U$3G$3.PB5
- net +3V3: now also U$3G$1.VDDBU, U$3G$1.VDDIN, U$3G$1.VDDIO; no longer U$1G$1.VDDBU, U$1G$1.VDDIN, U$1G$1.VDDIO
- net +5V: now also C36.2, IC2.VCC, IC2.VCCIO, IC2._RESET, R26.2, R27.2, X1G41.1
- net FLASH_CS: now also U$3G$4.PC2; no longer U$1G$4.PC2
- net FLASH_HLD: now also U$3G$4.ERASE/PC9; no longer U$1G$4.ERASE/PC9
- net FLASH_MISO: now also U$3G$4.PC3; no longer U$1G$4.PC3
- net FLASH_MOSI: now also U$3G$4.PC4; no longer U$1G$4.PC4
- net FLASH_SCLK: now also U$3G$4.PC5
- net FLASH_WP: now also U$3G$4.PC8; no longer U$1G$4.PC8
- net GND: now also C36.1, C37.2, C38.1, C39.2, IC2.AGND, IC2.GND1, IC2.GND2, IC2.GND3, IC2.TEST, IC3.VSS, JP2.4, JP2.5, U$3G$1.GND, U5.CD2, U5.GND, U5.SHIELD@3, X1G41.4, X1G41.5; no longer C30.2, C31.1, U$1G$1.GND
- net N$11: now also U$3G$1.XIN32; no longer U$1G$1.XIN32
- net N$12: now also U$3G$1.XOUT32; no longer U$1G$1.XOUT32
- net N$16: now also U$3G$2.PA29; no longer U$1G$2.PA29
- net N$17: now also U$3G$2.PA31; no longer U$1G$2.PA31
- net NRST: now also U$3G$1.NRST; no longer U$1G$1.NRST
- net SD_SPI_CS: now also U$3G$2.PA5/AD5; no longer U$1G$2.PA5/AD2
- net SD_SPI_DI: now also U$3G$2.PA7; no longer U$1G$2.PA7
- net SD_SPI_DO: now also U$3G$2.PA6; no longer U$1G$2.PA6
- net SD_SPI_SCK: now also U$3G$2.PA8; no longer U$1G$2.PA8
- net TCK: now also U$3G$3.TCK/SWCLK/PB3; no longer U$1G$3.PB3/TCK/SWCLK
- net TDI: now also U$3G$3.TDI/PB0; no longer U$1G$3.PB0/TWD1/TDI
- net TDO: now also U$3G$3.TDO/TRACESWO/PB1/RTOUT0; no longer U$1G$3.PB1/TWCK1/TDO/TRACESWO
- net TMS: now also U$3G$3.TMS/SWDIO/PB2; no longer U$1G$3.PB2/TMS/SWDIO
- net VDDLCD: no longer U$1G$1.VDDLCD
- net VDDOUT: now also U$3G$1.VDDCORE, U$3G$1.VDDOUT, U$3G$1.VDDPLL; no longer U$1G$1.VDDCORE, U$1G$1.VDDOUT, U$1G$1.VDDPLL
Other:
- note added: "Optional Debug Header"

Commit message: Started Layout - Pushing incase of act of God
Like fire, lighting strike, armageddon
Parts:
- removed C12: (no value), adafruit:C-USC0805
- removed C36: 10nF, passives:C0603
- removed IC3: MS25P05-A, OBD-Interface:MS25P05-A
- removed R24, R25: 0R, passives:R0603
- added C30, C31, C34: 100 nF, passives:C0603
Connections:
- removed net 2.8V: Q3.D, R9.2
- removed net FLASH_CS: IC3.CS, U$3G$4.PC2
- removed net FLASH_HLD: IC3.HLD, U$3G$4.ERASE/PC9
- removed net FLASH_MISO: IC3.MISO, U$3G$4.PC3
- removed net FLASH_MOSI: IC3.MOSI, U$3G$4.PC4
- removed net FLASH_SCLK: IC3.SCLK, U$3G$4.PC5
- removed net FLASH_WP: IC3.WP, U$3G$4.PC8
- removed net N$16: R24.1, U$3G$2.PA29
- removed net N$17: R25.1, U$3G$2.PA31
- removed net N$37: JP3.6, U$3G$3.PB17
- removed net VBAT: C9.1, IC4.IN
- net !VPW_RX: now also U$3G$3.PB31/AD5
- net +12V: now also C9.1, IC4.IN
- net +3V3: no longer IC3.VCC
- net +5V: no longer C12.1, C36.2, X1G41.1
- net 5/7V: now also Q3.D, R9.2
- net GND: now also C30.2, C31.2, C34.2, JP3.6; no longer C12.2, C36.1, IC3.VSS
- net N$18: now also U$3G$2.PA31; no longer R25.2
- net N$22: now also U$3G$2.PA29; no longer R24.2
- net PWM/!VPW: now also U$3G$3.PB29
- net VDDLCD: now also U$3G$1.VDDLCD
- net VDDOUT: now also C30.1, C31.1, C34.1
Other:
- note removed: "M25P05-AVMN6TP FLASH"

Commit message: More
Parts:
- removed C30, C31, C34: 100 nF, passives:C0603
- removed R23: 0 (NOPOP), passives:R0603
- added C12: (no value), adafruit:C-USC0805
Connections:
- removed net +12V: C1.1, C9.1, IC1.RUN1, IC1.RUN2, IC1.VIN1, IC1.VIN1_2, IC1.VIN2, IC1.VIN2_2, IC4.IN, JP2.16
- removed net N$19: JP1.15, R23.1
- new net VIN: C1.1, C12.1, C9.1, IC1.RUN1, IC1.RUN2, IC1.VIN1, IC1.VIN1_2, IC1.VIN2, IC1.VIN2_2, IC4.IN, JP2.16
- net GND: now also C12.2; no longer C30.2, C31.2, C34.2
- net NRST: now also JP1.15; no longer R23.2
- net VDDOUT: no longer C30.1, C31.1, C34.1
Other:
- moved on the sheet: C29
Changed lines of the file:
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@@
 <part name="R21" library="passives" deviceset="R" device="0603" value="100k"/>
 <part name="R22" library="passives" deviceset="R" device="0603" value="100k"/>
-<part name="R23" library="passives" deviceset="R" device="0603" value="0 (NOPOP)"/>
 <part name="U5" library="SparkFun-Connectors" deviceset="USD-SOCKET" device="USD"/>
 <part name="GND11" library="supply1" deviceset="GND" device=""/>
@@
 <part name="JP3" library="adafruit" deviceset="PINHD-1X6" device="CLEAN"/>
 <part name="U$3" library="OBD-Interface" deviceset="SAM4C32C-100" device=""/>
-<part name="C30" library="passives" deviceset="C" device="0603" value="100 nF"/>
-<part name="C31" library="passives" deviceset="C" device="0603" value="100 nF"/>
-<part name="C34" library="passives" deviceset="C" device="0603" value="100 nF"/>
 <part name="GND24" library="supply1" deviceset="GND" device=""/>
+<part name="C12" library="adafruit" deviceset="C-US" device="C0805"/>
+<part name="GND28" library="supply1" deviceset="GND" device=""/>
 </parts>
 <sheets>
@@
 <instance part="C27" gate="A" x="50.8" y="-10.16" rot="R270"/>
 <instance part="C28" gate="A" x="55.88" y="-10.16" rot="R270"/>
-<instance part="C29" gate="A" x="60.96" y="-10.16" rot="R270"/>
-<instance part="GND26" gate="1" x="60.96" y="-20.32"/>
+<instance part="C29" gate="A" x="63.5" y="-10.16" rot="R270"/>
+<instance part="GND26" gate="1" x="63.5" y="-20.32"/>
 <instance part="JP1" gate="G$1" x="185.42" y="-20.32" rot="MR0"/>
 <instance part="+3V3" gate="G$1" x="175.26" y="2.54"/>
@@
 <instance part="R21" gate="A" x="215.9" y="-7.62" rot="R90"/>
 <instance part="R22" gate="A" x="220.98" y="-7.62" rot="R90"/>
-<instance part="R23" gate="A" x="208.28" y="-27.94"/>
 <instance part="U$3" gate="G$1" x="-12.7" y="-20.32"/>
-<instance part="C30" gate="A" x="60.96" y="-10.16" rot="R270"/>
-<instance part="C31" gate="A" x="60.96" y="-10.16" rot="R270"/>
-<instance part="C34" gate="A" x="60.96" y="-10.16" rot="R270"/>
+<instance part="C12" gate="G$1" x="27.94" y="104.14"/>
+<instance part="GND28" gate="1" x="27.94" y="91.44"/>
 </instances>
 <busses>
@@
 <wire x1="45.72" y1="-15.24" x2="50.8" y2="-15.24" width="0.1524" layer="91"/>
 <wire x1="50.8" y1="-15.24" x2="55.88" y2="-15.24" width="0.1524" layer="91"/>
-<wire x1="55.88" y1="-15.24" x2="60.96" y2="-15.24" width="0.1524" layer="91"/>
-<wire x1="60.96" y1="-15.24" x2="60.96" y2="-12.7" width="0.1524" layer="91"/>
+<wire x1="55.88" y1="-15.24" x2="63.5" y2="-15.24" width="0.1524" layer="91"/>
 <pinref part="C28" gate="A" pin="2"/>
 <wire x1="55.88" y1="-12.7" x2="55.88" y2="-15.24" width="0.1524" layer="91"/>
@@
 <pinref part="C24" gate="A" pin="2"/>
 <wire x1="30.48" y1="-12.7" x2="30.48" y2="-15.24" width="0.1524" layer="91"/>
-<wire x1="60.96" y1="-15.24" x2="60.96" y2="-17.78" width="0.1524" layer="91"/>
+<wire x1="63.5" y1="-15.24" x2="63.5" y2="-17.78" width="0.1524" layer="91"/>
 <pinref part="GND26" gate="1" pin="GND"/>
 <junction x="30.48" y="-15.24"/>
@@
 <junction x="50.8" y="-15.24"/>
 <junction x="55.88" y="-15.24"/>
-<pinref part="C30" gate="A" pin="2"/>
-<junction x="60.96" y="-12.7"/>
-<pinref part="C31" gate="A" pin="2"/>
-<pinref part="C34" gate="A" pin="2"/>
+<wire x1="63.5" y1="-15.24" x2="63.5" y2="-12.7" width="0.1524" layer="91"/>
 </segment>
 <segment>
@@
 <junction x="175.26" y="-17.78"/>
 <junction x="175.26" y="-15.24"/>
+</segment>
+<segment>
+<pinref part="C12" gate="G$1" pin="2"/>
+<pinref part="GND28" gate="1" pin="GND"/>
+<wire x1="27.94" y1="99.06" x2="27.94" y2="93.98" width="0.1524" layer="91"/>
 </segment>
 </net>
@@
 </segment>
 </net>
-<net name="+12V" class="0">
+<net name="VIN" class="0">
 <segment>
 <pinref part="IC1" gate="A" pin="VIN1_2"/>
@@
 <wire x1="60.96" y1="119.38" x2="50.8" y2="129.54" width="0.1524" layer="91"/>
 <junction x="50.8" y="129.54"/>
-<wire x1="38.1" y1="129.54" x2="22.86" y2="129.54" width="0.1524" layer="91"/>
+<wire x1="38.1" y1="129.54" x2="27.94" y2="129.54" width="0.1524" layer="91"/>
 <junction x="38.1" y="129.54"/>
 <pinref part="P+2" gate="1" pin="+12V"/>
+<pinref part="C12" gate="G$1" pin="1"/>
+<wire x1="27.94" y1="129.54" x2="22.86" y2="129.54" width="0.1524" layer="91"/>
+<wire x1="27.94" y1="106.68" x2="27.94" y2="129.54" width="0.1524" layer="91"/>
+<junction x="27.94" y="129.54"/>
 </segment>
 </net>
@@
 <wire x1="45.72" y1="-5.08" x2="50.8" y2="-5.08" width="0.1524" layer="91"/>
 <wire x1="50.8" y1="-5.08" x2="55.88" y2="-5.08" width="0.1524" layer="91"/>
-<wire x1="55.88" y1="-5.08" x2="60.96" y2="-5.08" width="0.1524" layer="91"/>
-<wire x1="60.96" y1="-5.08" x2="60.96" y2="-7.62" width="0.1524" layer="91"/>
+<wire x1="55.88" y1="-5.08" x2="63.5" y2="-5.08" width="0.1524" layer="91"/>
 <pinref part="C23" gate="A" pin="1"/>
 <wire x1="25.4" y1="-7.62" x2="25.4" y2="-5.08" width="0.1524" layer="91"/>
@@
 <pinref part="U$3" gate="G$1" pin="VDDOUT"/>
 <pinref part="U$3" gate="G$1" pin="VDDPLL"/>
-<pinref part="C30" gate="A" pin="1"/>
-<junction x="60.96" y="-7.62"/>
-<pinref part="C31" gate="A" pin="1"/>
-<pinref part="C34" gate="A" pin="1"/>
+<wire x1="63.5" y1="-5.08" x2="63.5" y2="-7.62" width="0.1524" layer="91"/>
 </segment>
 </net>
@@
 <wire x1="220.98" y1="-27.94" x2="220.98" y2="-10.16" width="0.1524" layer="91"/>
 <wire x1="220.98" y1="-27.94" x2="231.14" y2="-27.94" width="0.1524" layer="91"/>
-<pinref part="R23" gate="A" pin="2"/>
-<wire x1="210.82" y1="-27.94" x2="220.98" y2="-27.94" width="0.1524" layer="91"/>
 <junction x="220.98" y="-27.94"/>
 <label x="231.14" y="-27.94" size="1.27" layer="95" xref="yes"/>
+<pinref part="JP1" gate="G$1" pin="15"/>
+<wire x1="193.04" y1="-27.94" x2="220.98" y2="-27.94" width="0.1524" layer="91"/>
 </segment>
 <segment>
@@
 <junction x="10.16" y="-30.48"/>
 <pinref part="U$3" gate="G$1" pin="NRST"/>
-</segment>
-</net>
-<net name="N$19" class="0">
-<segment>
-<pinref part="JP1" gate="G$1" pin="15"/>
-<pinref part="R23" gate="A" pin="1"/>
-<wire x1="193.04" y1="-27.94" x2="205.74" y2="-27.94" width="0.1524" layer="91"/>
 </segment>
 </net>
@@
 </segment>
 </net>
-<net name="+12V" class="0">
+<net name="VIN" class="0">
 <segment>
 <pinref part="JP2" gate="G$1" pin="16"/>
@@
 </segment>
 </net>
-<net name="+12V" class="0">
+<net name="VIN" class="0">
 <segment>
 <pinref part="C9" gate="G$1" pin="1"/>
