File: Hardware/Eagle Files/OBD-Interface/OBD-Schematic.brd (EAGLE design)
At the start: 160 x 100 mm, 86 parts, among them IC1 LTC3633EUFDPBF, IC2 FT232RL, IC3 MS25P05-A, IC4 V_REG_317DPACK, IC5 MCP2551, Q1 BSS138, Q2 BSS138, Q3 ZXMP6A13FTA, U3 LM339, U5 USD-SOCKETUSD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

Commit message: Started Layout - Pushing incase of act of God
Like fire, lighting strike, armageddon
Parts:
- removed C12: (no value), adafruit:C0805
- removed C36: 10nF, passives:C0603
- removed IC3: MS25P05-A, OBD-Interface:SO-08
- removed R24, R25: 0R, passives:R0603
- added C30, C31, C34: 100 nF, passives:C0603
- moved R27 160.8 mm to (72.4, 31.8)
- moved C38 156.7 mm to (72.4, 27.9), turned to 270 degrees
- moved C37 155.5 mm to (76.2, 27.9), turned to 90 degrees
- moved R26 155.2 mm to (72.4, 34.3)
- moved C33 148.0 mm to (59.7, 1.27), turned to 180 degrees
- moved R8 144.8 mm to (72.4, 36.8)
- moved LED1 142.3 mm to (77.5, 36.8), turned to 270 degrees
- moved C32 137.4 mm to (52.1, 1.27)
- moved C18 136.9 mm to (42.5, 11.4), turned to 270 degrees
- moved C13 136.4 mm to (38.7, 11.4), turned to 270 degrees
- moved C25 131.9 mm to (46.4, 11.4), turned to 270 degrees
- moved Y2CTX900-ND 129.3 mm to (55.9, 6.35), turned to 180 degrees
- moved C39 128.9 mm to (72.4, 39.4)
- moved R14 128.6 mm to (53.3, 34.3)
- moved C5 127.5 mm to (46.4, 36.8), turned to 90 degrees
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Connections:
- removed net 2.8V: Q3.3, R9.2
- removed net FLASH_CS: IC3.1, U$3.58
- removed net FLASH_HLD: IC3.7, U$3.29
- removed net FLASH_MISO: IC3.2, U$3.57
- removed net FLASH_MOSI: IC3.5, U$3.56
- removed net FLASH_SCLK: IC3.6, U$3.55
- removed net FLASH_WP: IC3.3, U$3.54
- removed net N$16: R24.1, U$3.59
- removed net N$17: R25.1, U$3.51
- removed net N$37: JP3.6, U$3.97
- removed net VBAT: C9.1, IC4.3
- net !VPW_RX: now also U$3.79
- net +12V: now also C9.1, IC4.3
- net +3V3: no longer IC3.8
- net +5V: no longer C12.1, C36.2, X1.1
- net 5/7V: now also Q3.3, R9.2
- net GND: now also C30.2, C31.2, C34.2, JP3.6; no longer C12.2, C36.1, IC3.4
- net N$18: now also U$3.51; no longer R25.2
- net N$22: now also U$3.59; no longer R24.2
- net PWM/!VPW: now also U$3.12
- net VDDOUT: now also C30.1, C31.1, C34.1
Other:
- board size 160 x 100 mm -> 80.6 x 51.1 mm

Commit message: More
Parts:
- removed C30, C31, C34: 100 nF, passives:C0603
- removed R23: 0 (NOPOP), passives:R0603
- added C12: (no value), adafruit:C0805
- moved R18 114.4 mm to (67.3, 40.6), turned to 90 degrees
- moved R21 112.0 mm to (59.7, 40.6), turned to 90 degrees
- moved R19 111.8 mm to (64.8, 40.6), turned to 90 degrees
- moved R20 109.3 mm to (62.2, 40.6), turned to 90 degrees
- moved R22 104.4 mm to (57.1, 40.6), turned to 90 degrees
- moved C7 102.9 mm to (33.0, 17.8)
- moved C2 87.1 mm to (20.3, 19.7), turned to 90 degrees
- moved C4 84.7 mm to (20.3, 36.2), turned to 270 degrees
- moved C1 80.7 mm to (20.3, 30.5), turned to 90 degrees
- moved C3 76.4 mm to (12.1, 22.9), turned to 180 degrees
- moved C6 76.4 mm to (12.7, 33.0), turned to 180 degrees
- moved R3 56.2 mm to (3.81, 30.5), turned to 90 degrees
- moved R1 55.2 mm to (-1.27, 19.1), turned to 180 degrees
- moved R2 53.2 mm to (-1.27, 14.0), turned to 180 degrees
- moved R4 46.4 mm to (3.81, 36.8), turned to 90 degrees
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Connections:
- removed net +12V: C1.1, C9.1, IC1.15, IC1.16, IC1.21, IC1.22, IC1.3, IC1.6, IC4.3, JP2.16
- removed net N$19: JP1.15, R23.1
- new net VIN: C1.1, C12.1, C9.1, IC1.15, IC1.16, IC1.21, IC1.22, IC1.3, IC1.6, IC4.3, JP2.16
- net GND: now also C12.2; no longer C30.2, C31.2, C34.2
- net NRST: now also JP1.15; no longer R23.2
- net VDDOUT: no longer C30.1, C31.1, C34.1
Routing:
- added copper zone on layer 1, net +3V3
- added copper zone on layer 1, net +5V
- added copper zone on layer 1, net GND
- added copper zone on layer 1, net N$2
- added copper zone on layer 1, net SW1
- added copper zone on layer 1, net SW2
- added copper zone on layer 1, net VIN
Other:
- board size 80.6 x 51.1 mm -> 84.4 x 51.1 mm
